File: eagle/final-sprite/sprite.brd (EAGLE design)
At the start: 35 x 44.6 mm, 62 parts, among them P1 SPRITE_PIN, P2 SPRITE_PIN, U1 CC430F5137, U2 DRV8833CRTER, U3 DRV8833CRTER, X1 TCXO_7Z

Commit message: consistent board, pre-renumbering passives
Parts:
- removed C18: 10uF, rcl:C0402
- removed C19: 0.1uF, rcl:C0402
- removed JP2, JP3: (no value), SparkFun:1X02
- removed R18: (no value), resistor:R0402
- removed R25: 10K, rcl:R0402
- removed R26: 1K, rcl:R0402
- removed SUNSENSOR1, SUNSENSOR2: LIGHTSENSORALS, SparkFun-Sensors:ALS-PT19
- added C11: 100n, resistor:C0402
- added C12: 10n, resistor:C0402
- added R12, R13: (no value), resistor:R0402
- added TP1, TP2, TP3: TEST-POINT2, SparkFun-Connectors:PAD.02X.02
- C1: value 10uF -> 4.7u; device rcl:C0402 -> resistor:C0402
- C10, C2: value 2.2uF -> 2.2u
- C16: value (none) -> 10n
- C17: value (none) -> 10u
- C20, C22: value 0.1uF -> 0.1u
- C21, C8: value 10nF -> 10n
- C3: value 2.2nF -> 2.2n
- C4, C7: value 470nF -> 470n
- C5: value 10nF -> 0.1u; device SparkFun:0603-CAP -> resistor:C0402
- C6: value 100nF -> 4.7u; device SparkFun:0603-CAP -> resistor:C0402
- C9: value 10uF -> 10u
- R10, R9: value 1K -> OPT; device rcl:R0402 -> resistor:R0402
- R15: value (none) -> 750K
- R16: value (none) -> 910K
- R17: value (none) -> 130K
- R6: value 10K -> 442K; device rcl:R0402 -> resistor:R0402
- moved C6 359.7 mm to (-9.00, -326.4), turned to 0 degrees
- moved C5 355.7 mm to (-9.00, -322.4), turned to 0 degrees
- moved U3 150.9 mm to (29.3, 29.0)
- moved U$5 144.3 mm to (-1.76, -312.3)
- moved R6 115.0 mm to (-9.00, -331.3)
- moved R9 66.0 mm to (-9.00, -346.0)
- moved C1 58.0 mm to (-9.00, -318.4)
- moved R10 55.3 mm to (-9.00, -350.0)
Connections:
- net N$4 renamed VCORE
- removed net N$14: R10.2, U3.4
- removed net P2.0/A0: R6.2, SUNSENSOR1.E
- removed net P2.5/A5: R25.2, SUNSENSOR2.E
- new net DRDY: LSM9DS1.9, U1.11
- new net INT1: LSM9DS1.11, U1.3
- new net INT2: LSM9DS1.12, U1.4
- net COIL12_FAULT_B: no longer R9.1
- net COIL3_FAULT_B: no longer R26.1
- net GND: now also C11.2, C12.2, R13.1, R6.2; no longer C18.2, C19.2, R10.1, R25.1, R6.1
- net N$12: now also TP1.P$1
- net N$16: now also R6.1
- net N$7: now also LSM9DS1.13
- net REF: now also R12.2, R23.2; no longer R18.2
- net REG_D0: now also U1.15; no longer U1.3
- net REG_D1: now also U1.21; no longer U1.4
- net RST: no longer JP2.1
- net SCL: now also TP2.P$1
- net SDA: now also TP3.P$1
- net TERM: now also R12.1, R13.2; no longer R18.1, R23.2
- net TST: no longer JP2.2
- net UART_RX: no longer JP3.2
- net UART_TX: no longer JP3.1
- net VCC: now also C1.1, C5.1, R10.2, R9.1; no longer C18.1, C19.1, R26.2, R9.2, SUNSENSOR1.C, SUNSENSOR2.C
- net VCCA: now also C11.1, C12.1; no longer C5.1, C6.1
- net VCCINT: now also R9.2
- net VCCIO: now also C6.1, R10.1; no longer C1.1
Routing:
- net UART_TX: track 24.5 -> 10.3 mm
- net VCORE: track 9.82 -> 0.00 mm
- net UART_RX: track 25.0 -> 21.9 mm
- net RST: track 1.84 -> 0.00 mm

Commit message: Updated schematic with DRV8837 drivers
Parts:
- removed ANT-N, ANT-P: ANTENNA, SpriteAntenna:ANTENNA
- removed C20, C22: 0.1u, rcl:C0402
- removed C21: 10n, rcl:C0402
- removed LSM9DS1: LSM9DS1, SparkFun-Sensors:LGA24-8X4
- removed P1, P2: SPRITE_PIN, SpritePin:SPRITE_PIN
- removed R24: 10K, rcl:R0402
- removed S1, S2, S3, S4: TRISOLX-WING, TriSolX_QzQube:TRISOLX-T01
- removed U$1: UMAC, UMAC:UMAC
- removed U$5: LPS4018-223M, STAC:LPS4018-223M
- added A1, A2: SPRITEANTENNA_ANTENNA, STAC:SPRITEANTENNA_ANTENNA
- added B1: UMAC_UMAC, STAC:UMAC_UMAC
- added C13, C14: 4.7u, resistor:C0402
- added C15: 0.1u, resistor:C0402
- added D2, D3, D4: TRISOLX-WING, STAC:TRISOLX_QZQUBE_TRISOLX-T01
- added J1: M20-7910442R, STAC:M20-7910442R
- added L2: 12 nH, SparkFun:0603
- added LED1: (no value), SparkFun:LED-0603
- added R14: OPT, resistor:R0402
- added U4, U6, U7: DRV8837, STAC:SON50P200X200X75-8N
- added X2: SPRITEPIN_SPRITE_PIN, STAC:SPRITEPIN_SPRITE_PIN
- C1: value 4.7u -> 470n; device resistor:C0402 -> rcl:C0402
- C10: value 2.2u -> 100n; device rcl:C0402 -> resistor:C0402
- C11: value 100n -> 10n
- C12: value 10n -> 10u; device resistor:C0402 -> rcl:C0402
- C16: value 10n -> 2.2u; device resistor:C0402 -> rcl:C0402
- C2: value 2.2u -> 2.2n
- C3: value 2.2n -> 0.1u
- C4: value 470n -> 10n
- C5: device resistor:C0402 -> rcl:C0402
- C6: value 4.7u -> 10n; device resistor:C0402 -> rcl:C0402
- C8: value 10n -> 2.2u
- C9: value 10u -> 10n; device rcl:C0402 -> resistor:C0402
- D1: value (none) -> TRISOLX-WING; device SparkFun:LED-0603 -> STAC:TRISOLX_QZQUBE_TRISOLX-T01
- L1: value 12 nH -> LPS4018-223M; device SparkFun:0603 -> STAC:LPS4018-223M
- R1: value 15R -> 47K
- R10: value OPT -> 750K
- R11: value 1K -> 15R
- R12: value (none) -> 15R; device resistor:R0402 -> rcl:R0402
- R13: value (none) -> OPT
- R15: value 750K -> (none)
- R16: value 910K -> (none)
- R17: value 130K -> (none)
- R18, R19: value (none) -> 5M
- R2: value 56K -> 270R
- R20: value (none) -> 4.42M
- R21: value (none) -> 5.6M
- R22: value (none) -> 1K; device resistor:R0402 -> rcl:R0402
- R4: value 10K -> 56K
- R5: value 47K -> 10K
- R6: value 442K -> 10K; device resistor:R0402 -> rcl:R0402
- R7: value 270R -> 130K; device rcl:R0402 -> resistor:R0402
- R8: value 15R -> 910K; device rcl:R0402 -> resistor:R0402
- R9: value OPT -> 7K
- U1: value CC430F5137 -> CC430F513X; device TI_MSP430_v16:RGZ48 -> STAC:TI_MSP430_V16_RGZ48
- U2: value DRV8833CRTER -> LSM9DS1; device STAC:RTE16_1P66X1P66 -> SparkFun-Sensors:LGA24-8X4
- U3: value DRV8833CRTER -> (none); device STAC:RTE16_1P66X1P66 -> STAC:SPRITETCXO_TXC_7Z
- X1: value TCXO_7Z -> SPRITEPIN_SPRITE_PIN; device SpriteTCXO:TXC_7Z -> STAC:SPRITEPIN_SPRITE_PIN
- moved U1 499.8 mm to (-2.10, -473.6), turned to 0 degrees
- moved U3 496.5 mm to (-9.00, -466.0)
- moved D1 457.7 mm to (16.4, -427.6)
- moved L1 345.0 mm to (-1.76, -312.3), turned to 0 degrees
- moved R10 217.3 mm to (-5.90, -132.7)
- moved R20 198.2 mm to (-9.00, -354.9)
- moved R21 198.2 mm to (-9.00, -358.9)
- moved R8 138.4 mm to (-5.90, -136.7)
- moved R22 134.9 mm to (-9.30, -299.6)
- moved C5 125.7 mm to (-9.00, -196.7)
- moved C16 113.1 mm to (-9.00, -289.8)
- moved C9 108.2 mm to (-9.00, -176.7)
- moved C1 92.3 mm to (-9.00, -226.1)
- moved R7 90.4 mm to (-5.90, -140.7)
- moved R12 89.6 mm to (-9.30, -265.3)
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- renumbered R23 to R18, U$4 to U5
Connections:
- removed net COIL12_EN: U1.16, U2.15
- removed net COIL1_IN1: U1.20, U2.14
- removed net COIL1_IN2: U1.19, U2.13
- removed net COIL2_IN1: U1.18, U2.7
- removed net COIL2_IN2: U1.17, U2.8
- removed net COIL3_EN: U1.48, U3.15
- removed net COIL3_IN1: U1.2, U3.14
- removed net COIL3_IN2: U1.1, U3.13
- removed net N$10: R1.2, U2.1
- removed net N$15: R11.2, U3.1
- removed net N$9: R8.2, U2.4
- removed net VID: U1.23
- new net EN_1: U1.19, U4.7
- new net EN_2: U1.20, U6.7
- new net EN_3: U1.21, U7.7
- new net N$14: U4.3
- new net N$26: R12.1, U6.2
- new net N$27: U6.3
- new net N$28: U7.3
- new net PWM1: U1.17, U4.6, U6.6, U7.6
- new net PWM2: U1.18, U4.5, U6.5, U7.5
- new net VSYS: C14.1, C15.1, R13.2, R14.1, U5.16
- net COIL12_FAULT_B: no longer U2.6
- net COIL3_FAULT_B: no longer U3.6
- net DRDY: now also U2.9; no longer LSM9DS1.9
- net GND: now also B1.V-, C13.2, C14.2, C15.2, C2.1, C3.2, C8.2, D1.P$3, D2.P$3, D3.P$3, D4.P$3, J1.6, LED1.C, R10.1, R17.1, R21.1, R4.1, R9.2, U2.14, U2.15, U2.16, U2.18, U2.19, U2.20, U3.GND1, U3.GND2, U4.4, U4.9, U6.4, U6.9, U7.4, U7.9, X2.PIN; no longer C2.2, C20.2, C21.2, C22.2, C3.1, C6.2, D1.C, LSM9DS1.14, LSM9DS1.15, LSM9DS1.16, LSM9DS1.17, LSM9DS1.18, LSM9DS1.19, LSM9DS1.20, P2.PIN, R1.1, R11.1, R13.1, R15.1, R16.1, R2.1, R22.1, R6.2, S1.P$3, S2.P$3, S3.P$3, S4.P$3, U$1.V-, U2.11, U3.11, U3.17, X1.GND1, X1.GND2
- net INT1: now also U2.11; no longer LSM9DS1.11
- net INT2: now also U2.12; no longer LSM9DS1.12
- net N$1: now also C6.1; no longer C8.1
- net N$11: now also LED1.A, R2.1; no longer D1.A, R7.1
- net N$12: now also C6.2, U3.OUT; no longer C8.2, X1.OUT
- net N$13: now also R22.1, U7.2; no longer C10.1, U3.12
- net N$16: now also R9.1; no longer R24.1, R6.1
- net N$18: now also R7.1, R8.2; no longer R16.2, R17.1
- net N$2: now also R2.2; no longer R7.2
- net N$20: now also R10.2; no longer R15.2
- net N$21: now also C9.1; no longer C16.1
- net N$22: now also L1.P$2; no longer U$5.P$2
- net N$3: now also R4.2; no longer R2.2
- net N$5: now also C5.1, U2.24; no longer C22.1, LSM9DS1.24
- net N$6: now also C4.1, U2.21; no longer C21.1, LSM9DS1.21
- net N$7: now also R6.2, U2.13, U2.5, U2.6, U2.7, U2.8; no longer LSM9DS1.13, LSM9DS1.5, LSM9DS1.6, LSM9DS1.7, LSM9DS1.8, R24.1
- net N$8: now also R11.1, U4.2; no longer C2.1, U2.12
- net REF: now also R15.2; no longer R12.2
- net REG_D1: now also U1.16; no longer U1.21
- net RF_N: now also A1.IN1, A1.IN2, A1.IN3; no longer ANT-N.IN1, ANT-N.IN2, ANT-N.IN3
- net RF_P: now also A2.IN1, A2.IN2, A2.IN3; no longer ANT-P.IN1, ANT-P.IN2, ANT-P.IN3
- net RST: now also C2.2, J1.2, R1.1; no longer C3.2, R5.1
- net SCL: now also R5.1, U2.2; no longer LSM9DS1.2, R4.1
- net SDA: now also U2.4; no longer LSM9DS1.4
- net SETHYS: now also R16.1, R17.2; no longer R21.1, R22.2
- net SETPG: now also R15.1, R16.2; no longer R20.1, R21.2
- net TERM: now also R20.1, R21.2; no longer R12.1, R13.2
- net TST: now also J1.3
- net UART_RX: now also J1.5
- net UART_TX: now also J1.4
- net VBAT: now also B1.V+; no longer U$1.V+
- net VCC: now also C3.1, C7.1, J1.1, L2.1, R1.2, R6.1, U2.1, U2.22, U2.23, U2.3, U4.8, U6.8, U7.8, X1.PIN; no longer C1.1, C20.1, C4.1, C5.1, L1.1, LSM9DS1.1, LSM9DS1.22, LSM9DS1.23, LSM9DS1.3, P1.PIN, R10.2, R24.2, R4.2, R9.1, U5.16, X1.VCC
- net VCCA: now also C10.1, L2.2, U3.VCC; no longer C12.1, L1.2
- net VCCINT: now also D1.P$2, D2.P$2, D3.P$2, D4.P$2, L1.P$1, R14.2, R7.2; no longer R17.2, R9.2, S1.P$2, S2.P$2, S3.P$2, S4.P$2, U$5.P$1
- net VCCIO: now also C12.1, C13.1, C16.1, C8.1, R13.1, U4.1, U6.1, U7.1; no longer C6.1, C9.1, R10.1, U2.10, U3.10
- net VCORE: now also C1.1; no longer C7.1
Routing:
- net VCCINT: track 23.3 -> 0.00 mm, vias 1 -> 0
- net UART_RX: track 21.9 -> 0.00 mm
- net GND: track 22.5 -> 2.92 mm, vias 4 -> 1
- net UART_TX: track 10.3 -> 0.00 mm
- net VCCA: track 7.66 -> 1.70 mm, vias 2 -> 0
- net N$3: track 4.41 -> 0.00 mm
- net RF_N: track 3.52 -> 0.00 mm
- net RF_P: track 3.31 -> 0.00 mm
- net N$2: track 1.16 -> 0.00 mm
- net VCC: track 0.85 -> 0.00 mm
- net N$1: track 0.83 -> 0.00 mm

Commit message: Remove unused fault nets
Connections:
- removed net COIL12_FAULT_B: U1.13
- removed net COIL3_FAULT_B: U1.12
Changed lines of the file:
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@@
 <?xml version="1.0" encoding="utf-8"?>
 <!DOCTYPE eagle SYSTEM "eagle.dtd">
-<eagle version="9.0.1">
+<eagle version="9.0.0">
 <drawing>
 <settings>
@@
 <wire x1="-0.82" y1="-90.65" x2="-0.82" y2="-91.15" width="0" layer="19" extent="1-1"/>
 </signal>
-<signal name="COIL12_FAULT_B">
-<contactref element="U1" pad="13"/>
-</signal>
-<signal name="COIL3_FAULT_B">
-<contactref element="U1" pad="12"/>
-</signal>
 <signal name="REG_D0">

Commit message: started layout and fixed R0402 packages
Parts:
- R1, R11, R12, R2, R3, R4, R5, R6: device rcl:R0402 -> resistor:R0402
- R22: value 1K -> 15R; device rcl:R0402 -> resistor:R0402
- moved U1 499.8 mm to (8.30, 26.1), turned to 135 degrees
- moved J1 494.0 mm to (1.70, 11.4), turned to 270 degrees
- moved D4 492.8 mm to (20.3, 31.0), flipped to the bottom, turned to 90 degrees
- moved U3 491.6 mm to (1.70, 25.5), turned to 90 degrees
- moved D3 456.6 mm to (19.9, 6.20), flipped to the bottom, turned to 270 degrees
- moved D2 454.0 mm to (30.1, 14.8)
- moved D1 442.1 mm to (7.30, 14.4), turned to 180 degrees
- moved A2 431.2 mm to (2.30, 30.0), turned to 10 degrees
- moved A1 421.3 mm to (5.00, 32.7), turned to 80 degrees
- moved C11 371.9 mm to (13.2, 30.1)
- moved C10 365.5 mm to (13.3, 28.6)
- moved R3 310.7 mm to (-9.30, -517.2)
- moved R5 310.7 mm to (-9.30, -522.1)
- moved R2 296.0 mm to (-9.30, -527.0)
- moved R1 296.0 mm to (-9.30, -536.8)
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Connections:
- net GND: now also R4.2; no longer R4.1
- net N$11: now also R2.2; no longer R2.1
- net N$2: now also R2.1; no longer R2.2
- net N$3: now also R4.1; no longer R4.2
- net RST: now also R1.2; no longer R1.1
- net SCL: now also R3.2; no longer R5.1
- net SDA: now also R5.2; no longer R3.1
- net VCC: now also R1.1, R3.1, R5.1; no longer R1.2, R3.2, R5.2

Commit message: some schematic updates
Parts:
- added L3, L4: PCBSAT-TORQUECOIL, STAC:PCBSAT-TORQUECOIL
- R18: value 5M -> 5.49M
- R19: value 5M -> 4.53M
Connections:
- new net N$4: L3.1, R11.2
- new net N$9: L4.1, R12.2
- net N$14: now also L3.2
- net N$27: now also L4.2
- net N$28: now also R22.2
Changed lines of the file:
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@@
 <element name="R8" library="resistor" library_urn="urn:adsk.eagle:library:348" package="R0402" package3d_urn="urn:adsk.eagle:package:26058/1" value="910K" x="-5.9" y="-136.7"/>
 <element name="R7" library="resistor" library_urn="urn:adsk.eagle:library:348" package="R0402" package3d_urn="urn:adsk.eagle:package:26058/1" value="130K" x="-5.9" y="-140.7"/>
-<element name="R19" library="resistor" library_urn="urn:adsk.eagle:library:348" package="R0402" package3d_urn="urn:adsk.eagle:package:26058/1" value="5M" x="-5.9" y="-152.7"/>
+<element name="R19" library="resistor" library_urn="urn:adsk.eagle:library:348" package="R0402" package3d_urn="urn:adsk.eagle:package:26058/1" value="4.53M" x="-5.9" y="-152.7"/>
 <element name="R15" library="resistor" library_urn="urn:adsk.eagle:library:348" package="R0402" package3d_urn="urn:adsk.eagle:package:26058/1" value="" x="-5.9" y="-156.7"/>
 <element name="R16" library="resistor" library_urn="urn:adsk.eagle:library:348" package="R0402" package3d_urn="urn:adsk.eagle:package:26058/1" value="" x="-5.9" y="-160.7"/>
 <element name="R17" library="resistor" library_urn="urn:adsk.eagle:library:348" package="R0402" package3d_urn="urn:adsk.eagle:package:26058/1" value="" x="-5.9" y="-164.7"/>
-<element name="R18" library="resistor" library_urn="urn:adsk.eagle:library:348" package="R0402" package3d_urn="urn:adsk.eagle:package:26058/1" value="5M" x="-5.9" y="-168.7"/>
+<element name="R18" library="resistor" library_urn="urn:adsk.eagle:library:348" package="R0402" package3d_urn="urn:adsk.eagle:package:26058/1" value="5.49M" x="-5.9" y="-168.7"/>
 <element name="L1" library="STAC" package="LPS4018-223M" value="LPS4018-223M" x="-1.765" y="-312.3"/>
 <element name="C17" library="resistor" library_urn="urn:adsk.eagle:library:348" package="C0402" package3d_urn="urn:adsk.eagle:package:26136/1" value="10u" x="-9" y="-172.7"/>
@@
 <element name="R12" library="resistor" library_urn="urn:adsk.eagle:library:348" package="R0402" package3d_urn="urn:adsk.eagle:package:26058/1" value="15R" x="-9.3" y="-551.5"/>
 <element name="R22" library="resistor" library_urn="urn:adsk.eagle:library:348" package="R0402" package3d_urn="urn:adsk.eagle:package:26058/1" value="15R" x="-9.3" y="-556.4"/>
+<element name="L3" library="STAC" package="PCBSAT-TORQUECOIL" value="PCBSAT-TORQUECOIL" x="0.3" y="-563.7"/>
+<element name="L4" library="STAC" package="PCBSAT-TORQUECOIL" value="PCBSAT-TORQUECOIL" x="0.3" y="-573.1"/>
 </elements>
 <signals>
@@
 <signal name="N$14">
 <contactref element="U4" pad="3"/>
+<contactref element="L3" pad="2"/>
+<wire x1="5.3" y1="-560.7" x2="-9.385" y2="-489.45" width="0" layer="19" extent="1-1"/>
 </signal>
 <signal name="N$26">
@@
 <signal name="N$27">
 <contactref element="U6" pad="3"/>
+<contactref element="L4" pad="2"/>
+<wire x1="5.3" y1="-570.1" x2="-9.385" y2="-495.75" width="0" layer="19" extent="1-1"/>
 </signal>
 <signal name="N$13">
@@
 <signal name="N$28">
 <contactref element="U7" pad="3"/>
+<contactref element="R22" pad="2"/>
+<wire x1="-9.385" y1="-502.05" x2="-8.65" y2="-556.4" width="0" layer="19" extent="1-1"/>
 </signal>
 <signal name="VCCA">
@@
 <wire x1="-0.82" y1="-90.15" x2="-9.65" y2="-318.4" width="0" layer="19" extent="1-1"/>
 </signal>
+<signal name="N$4">
+<contactref element="L3" pad="1"/>
+<contactref element="R11" pad="2"/>
+<wire x1="-8.65" y1="-546.6" x2="-4.7" y2="-560.7" width="0" layer="19" extent="1-1"/>
+</signal>
+<signal name="N$9">
+<contactref element="L4" pad="1"/>
+<contactref element="R12" pad="2"/>
+<wire x1="-8.65" y1="-551.5" x2="-4.7" y2="-570.1" width="0" layer="19" extent="1-1"/>
+</signal>
 </signals>

Commit message: Placed all components, probably
Parts:
- removed C16: 2.2u, rcl:C0402
- removed TP1, TP2, TP3: TEST-POINT2, SparkFun-Connectors:PAD.02X.02
- C8: value 2.2u -> 10u
- moved L4 607.1 mm to (20.4, 33.7), flipped to the bottom
- moved R12 581.7 mm to (32.8, 28.7), flipped to the bottom, turned to 90 degrees
- moved L3 577.7 mm to (1.30, 14.0), flipped to the bottom, turned to 270 degrees
- moved R22 567.2 mm to (29.0, 9.50), flipped to the bottom
- moved R4 559.5 mm to (1.70, 27.5), turned to 180 degrees
- moved R1 558.4 mm to (2.30, 21.5)
- moved R5 555.3 mm to (23.4, 32.2), turned to 270 degrees
- moved R2 554.9 mm to (16.5, 27.3)
- moved R11 552.8 mm to (4.80, 6.00), turned to 270 degrees
- moved R3 550.6 mm to (27.1, 32.2), turned to 270 degrees
- moved R6 545.6 mm to (25.2, 32.2), turned to 270 degrees
- moved U7 507.8 mm to (6.90, 5.80), flipped to the bottom
- moved U6 507.0 mm to (6.90, 11.3), flipped to the bottom, turned to 180 degrees
- moved U4 499.8 mm to (3.60, 10.5), turned to 90 degrees
- moved R21 379.2 mm to (9.40, 19.9), flipped to the bottom, turned to 270 degrees
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Connections:
- net GND: no longer C16.2
- net N$12: no longer TP1.P$1
- net PWM1: now also U1.1; no longer U1.17
- net PWM2: now also U1.2; no longer U1.18
- net SCL: no longer TP2.P$1
- net SDA: no longer TP3.P$1
- net VCCIO: no longer C16.1
Routing:
- net GND: track 2.92 -> 0.16 mm, vias 1 -> 0
- net VCCA: track 1.70 -> 0.00 mm
