File: kicad/final-sprite/sprite.sch (KiCad schematic (older format))
At the start: 64 parts, among them J1 M20-7910442R, U1 CC430F513X, U2 LSM9DS1, U3 SPRITETCXO_TCXO_7Z, U4 DRV8837, U5 ADP5092, U6 DRV8837, U7 DRV8837, X1 SPRITEPIN_SPRITE_PIN, X2 SPRITEPIN_SPRITE_PIN

Commit message: Fix inductor
Connections:
- net labels added: SWN
Changed lines of the file:
@@
 Wire Wire Line
 	9150 9600 9700 9600
+Text Label 8700 2800 0    50   ~ 0
+SWN
 $EndSCHEMATC

Commit message: Remove extra test point
Parts:
- removed TP1: Test_Point, TestPoint:TestPoint_Pad_D1.0mm, symbol Connector:Test_Point
Changed lines of the file:
@@
 Wire Wire Line
 	8850 9100 8850 9050
-$Comp
-L Connector:Test_Point TP1
-U 1 1 5B35E6CA
-P 8550 10000
-F 0 "TP1" H 8608 10120 50  0000 L CNN
-F 1 "Test_Point" H 8608 10029 50  0000 L CNN
-F 2 "TestPoint:TestPoint_Pad_D1.0mm" H 8750 10000 50  0001 C CNN
-F 3 "~" H 8750 10000 50  0001 C CNN
-	1    8550 10000
-	1    0    0    1
-$EndComp
 Wire Wire Line
 	9150 10000 8550 10000
 Wire Wire Line
 	8550 10000 8550 9200
-Connection ~ 8550 10000
 Wire Wire Line
 	8550 9200 9150 9200

Commit message: Fix footprints and layout
Parts:
- removed C10: 100n, sprite:C0402, symbol sprite-eagle-import:C-EUC0402
Connections:
- net labels added: ~RST
- net labels removed: RST
- wire segments 270 -> 267
Changed lines of the file:
@@
 	6400 7000 6400 6800
 Connection ~ 6400 7000
-Text Label 5000 7000 0    10   ~ 0
-VCC
 Wire Wire Line
 	5000 6300 5700 6300
@@
 GND
 Wire Wire Line
-	6200 10100 6200 10200
-Text Label 6200 10100 0    10   ~ 0
-GND
-Wire Wire Line
 	6500 10100 6500 10200
 Text Label 6500 10100 0    10   ~ 0
@@
 Wire Wire Line
 	10100 7500 10300 7500
-Text Label 10100 7500 0    10   ~ 0
-GND
 Wire Wire Line
 	9700 6600 9500 6600
@@
 	5000 6400 5300 6400
 Text Label 5025 6400 0    70   ~ 0
-RST
+~RST
 Wire Wire Line
 	1500 9800 1800 9800
@@
 	2000 9800 2400 9800
 Text Label 1500 9800 0    70   ~ 0
-RST
+~RST
 Connection ~ 2000 9800
 Connection ~ 1800 9800
@@
 VCCIO
 Wire Wire Line
-	8800 2400 8800 2100
-Wire Wire Line
 	8800 2100 8000 2100
 Text Label 8200 2100 0    70   ~ 0
@@
 	3200 7000 2700 7000
 Text Label 2700 7000 0    70   ~ 0
-REG_D0
+REG_D1
 Wire Wire Line
 	8800 2500 8700 2500
-Wire Wire Line
-	8700 2500 8700 2200
 Wire Wire Line
 	8700 2200 8000 2200
@@
 	3200 6800 2700 6800
 Text Label 2700 6800 0    70   ~ 0
-REG_D1
+REG_D0
 Wire Wire Line
 	7900 3800 7900 3400
@@
 Connection ~ 5400 7600
 Connection ~ 5400 7200
-Text Label 5000 7200 0    10   ~ 0
-VCCA
-Wire Wire Line
-	5900 9700 6200 9700
-Wire Wire Line
-	6200 9700 6200 9800
-Wire Wire Line
-	6200 9700 6500 9700
 Wire Wire Line
 	6500 9700 6500 9800
 Wire Wire Line
 	6500 9700 6500 9600
-Connection ~ 6200 9700
 Connection ~ 6500 9700
 Text Label 5900 9700 0    10   ~ 0
@@
 $EndComp
 $Comp
-L sprite-eagle-import:VCC #P+09
-U 1 0 B2DC4156A813F830
-P 6400 6800
-F 0 "#P+09" H 6400 6800 50  0001 C CNN
-F 1 "VCC" H 6360 6940 59  0000 L BNN
-F 2 "" H 6400 6800 50  0001 C CNN
-F 3 "" H 6400 6800 50  0001 C CNN
-	1    6400 6800
-	1    0    0    -1
-$EndComp
-$Comp
 L sprite-eagle-import:VCC #P+03
 U 1 0 4985FDE44F0D6BCD
@@
 $EndComp
 $Comp
-L sprite-eagle-import:GND #GND016
-U 1 0 C691AFEA4CC6CA08
-P 6200 10300
-F 0 "#GND016" H 6200 10300 50  0001 C CNN
-F 1 "GND" H 6100 10200 59  0000 L BNN
-F 2 "" H 6200 10300 50  0001 C CNN
-F 3 "" H 6200 10300 50  0001 C CNN
-	1    6200 10300
-	-1   0    0    -1
-$EndComp
-$Comp
 L sprite-eagle-import:LED0603 LED1
 U 1 0 F49A53E384EE1AB4
@@
 	1    8400 2400
 	-1   0    0    1
-$EndComp
-$Comp
-L sprite-eagle-import:C-EUC0402 C10
-U 1 0 6551BB3D2910DE9F
-P 6200 9900
-F 0 "C10" H 6260 9915 59  0000 L BNN
-F 1 "100n" H 6260 9715 59  0000 L BNN
-F 2 "sprite:C0402" H 6200 9900 50  0001 C CNN
-F 3 "" H 6200 9900 50  0001 C CNN
-	1    6200 9900
-	1    0    0    -1
 $EndComp
 $Comp
@@
 Text Label 8700 2800 0    50   ~ 0
 SWN
+Wire Wire Line
+	8700 2500 8700 2200
+Wire Wire Line
+	8800 2400 8800 2100
+$Comp
+L sprite-eagle-import:VCCA #U$?
+U 1 0 5B2CFFE1
+P 6400 6800
+F 0 "#U$?" H 6400 6800 50  0001 C CNN
+F 1 "VCCA" H 6400 6910 59  0000 C BNN
+F 2 "" H 6400 6800 50  0001 C CNN
+F 3 "" H 6400 6800 50  0001 C CNN
+	1    6400 6800
+	1    0    0    -1
+$EndComp
+Wire Wire Line
+	5900 9700 6500 9700
 $EndSCHEMATC

Commit message: more routes fixed, removed some vias
Connections:
- wire segments 267 -> 268
Changed lines of the file:
@@
-REGGOOD
-Wire Wire Line
-	5000 5700 5600 5700
-Text Label 5125 5700 0    70   ~ 0
 REGGOOD
 Wire Wire Line
@@
 	8800 2400 8800 2100
 $Comp
-L sprite-eagle-import:VCCA #U$?
+L sprite-eagle-import:VCCA #U$0101
 U 1 0 5B2CFFE1
 P 6400 6800
-F 0 "#U$?" H 6400 6800 50  0001 C CNN
+F 0 "#U$0101" H 6400 6800 50  0001 C CNN
 F 1 "VCCA" H 6400 6910 59  0000 C BNN
 F 2 "" H 6400 6800 50  0001 C CNN
@@
 Wire Wire Line
 	5900 9700 6500 9700
+Wire Wire Line
+	5000 6700 5300 6700
+Text Label 5000 6700 0    50   ~ 0
+REGGOOD
+Wire Wire Line
+	3200 6700 2700 6700
+Text Label 2700 6700 0    50   ~ 0
+PGOOD
 $EndSCHEMATC

Commit message: Fixing pgood renaming
Connections:
- wire segments 268 -> 267
Changed lines of the file:
@@
-PGOOD
-Wire Wire Line
-	3200 7200 2700 7200
-Text Label 2700 7200 0    70   ~ 0
 PGOOD
 Wire Wire Line

Commit message: Changed resistor values
Parts:
- R1: value 47K -> 43K
- R15: value R-US_R0402 -> 5.49M
- R16: value R-US_R0402 -> 450K
- R17: value R-US_R0402 -> 4.53M
- R18: value 5.49M -> 5M
- R19: value 4.53M -> 5M
- R7: value 130K -> 150K
- R8: value 910K -> 1M
Other:
- note added: "All Caps 3.3V\nExcept C21 (16V)\nAll Passives 0402 \nAll Passives (5%)\nExcept R4, R15 - R21 (1%) \nSubject to Change\nR2, R11, R12, R22\nR7, R8\nC3\nMPPT Max efficiency:\nR7/(R7 + R8) = 87%\nVsetsd: \n1V*(1+R18/R19) = 2V\nVbat_term:\n(3/2)V*(1+R20/R21) = 2.7V\nVsetpg_falling: \n1V*(1+(R15/(R16+R17))) = 2.102V\nVsetpg_rising:\n1V*(1+((R15+R16)/R17)) = 2.311V"
- note removed: "All Caps 3.3V\nExcept C21 (16V)\nAll Passives 0402 \nAll Passives (5%)\nExcept R4, R15 - R21 (1%) \nSubject to Change\nR2, R11, R12, R22\nR7, R8\nC3\nMPPT Max efficiency:\nR7/(R7 + R8) = 87%"
Changed lines of the file:
@@
 P 7900 4000
 F 0 "R8" H 7750 4059 59  0000 L BNN
-F 1 "910K" H 7750 3870 59  0000 L BNN
+F 1 "1M" H 7750 3870 59  0000 L BNN
 F 2 "sprite:R0402" H 7900 4000 50  0001 C CNN
 F 3 "" H 7900 4000 50  0001 C CNN
@@
 P 7900 3200
 F 0 "R7" H 7750 3259 59  0000 L BNN
-F 1 "130K" H 7750 3070 59  0000 L BNN
+F 1 "150K" H 7750 3070 59  0000 L BNN
 F 2 "sprite:R0402" H 7900 3200 50  0001 C CNN
 F 3 "" H 7900 3200 50  0001 C CNN
@@
 P 13200 4000
 F 0 "R19" H 13050 4059 59  0000 L BNN
-F 1 "4.53M" H 13050 3870 59  0000 L BNN
+F 1 "5M" H 13050 3870 59  0000 L BNN
 F 2 "sprite:R0402" H 13200 4000 50  0001 C CNN
 F 3 "" H 13200 4000 50  0001 C CNN
@@
 P 12800 2600
 F 0 "R15" H 12650 2659 59  0000 L BNN
-F 1 "R-US_R0402" H 12650 2470 59  0000 L BNN
+F 1 "5.49M" H 12650 2470 59  0000 L BNN
 F 2 "sprite:R0402" H 12800 2600 50  0001 C CNN
 F 3 "" H 12800 2600 50  0001 C CNN
@@
 P 12800 3300
 F 0 "R16" H 12650 3359 59  0000 L BNN
-F 1 "R-US_R0402" H 12650 3170 59  0000 L BNN
+F 1 "450K" H 12650 3170 59  0000 L BNN
 F 2 "sprite:R0402" H 12800 3300 50  0001 C CNN
 F 3 "" H 12800 3300 50  0001 C CNN
@@
 P 12800 4000
 F 0 "R17" H 12650 4059 59  0000 L BNN
-F 1 "R-US_R0402" H 12650 3870 59  0000 L BNN
+F 1 "4.53M" H 12650 3870 59  0000 L BNN
 F 2 "sprite:R0402" H 12800 4000 50  0001 C CNN
 F 3 "" H 12800 4000 50  0001 C CNN
@@
 P 13200 2600
 F 0 "R18" H 13050 2659 59  0000 L BNN
-F 1 "5.49M" H 13050 2470 59  0000 L BNN
+F 1 "5M" H 13050 2470 59  0000 L BNN
 F 2 "sprite:R0402" H 13200 2600 50  0001 C CNN
 F 3 "" H 13200 2600 50  0001 C CNN
@@
 P 1800 9600
 F 0 "R1" H 1650 9659 59  0000 L BNN
-F 1 "47K" H 1650 9470 59  0000 L BNN
+F 1 "43K" H 1650 9470 59  0000 L BNN
 F 2 "sprite:R0402" H 1800 9600 50  0001 C CNN
 F 3 "" H 1800 9600 50  0001 C CNN
@@
 Text Notes 5800 7500 0    59   ~ 0
 1% REQ
-Text Notes 12800 7800 0    127  ~ 0
-All Caps 3.3V\nExcept C21 (16V)\nAll Passives 0402 \nAll Passives (5%)\nExcept R4, R15 - R21 (1%) \nSubject to Change\nR2, R11, R12, R22\nR7, R8\nC3\nMPPT Max efficiency:\nR7/(R7 + R8) = 87%
+Text Notes 12550 9300 0    127  ~ 0
+All Caps 3.3V\nExcept C21 (16V)\nAll Passives 0402 \nAll Passives (5%)\nExcept R4, R15 - R21 (1%) \nSubject to Change\nR2, R11, R12, R22\nR7, R8\nC3\nMPPT Max efficiency:\nR7/(R7 + R8) = 87%\nVsetsd: \n1V*(1+R18/R19) = 2V\nVbat_term:\n(3/2)V*(1+R20/R21) = 2.7V\nVsetpg_falling: \n1V*(1+(R15/(R16+R17))) = 2.102V\nVsetpg_rising:\n1V*(1+((R15+R16)/R17)) = 2.311V
 Wire Notes Line
 	12200 9900 12200 4800

Commit message: updated resistitator values again
Parts:
- R16: value 450K -> 453K
Other:
- note added: "All Caps 3.3V\nExcept C21 (16V)\nAll Passives 0402 \nAll Passives (5%)\nExcept R4, R15 - R21 (1%) \nSubject to Change\nR2, R11, R12, R22\nR7, R8\nC3\nMPPT Max efficiency:\nR7/(R7 + R8) = 87%\nVsetsd: \n1V*(1+R18/R19) = 2V\nVbat_term:\n(3/2)V*(1+R20/R21) = 2.7V\nVsetpg_falling: \n1V*(1+(R15/(R16+R17))) = 2.102V\nVsetpg_rising:\n1V*(1+((R15+R16)/R17)) = 2.312V"
- note removed: "All Caps 3.3V\nExcept C21 (16V)\nAll Passives 0402 \nAll Passives (5%)\nExcept R4, R15 - R21 (1%) \nSubject to Change\nR2, R11, R12, R22\nR7, R8\nC3\nMPPT Max efficiency:\nR7/(R7 + R8) = 87%\nVsetsd: \n1V*(1+R18/R19) = 2V\nVbat_term:\n(3/2)V*(1+R20/R21) = 2.7V\nVsetpg_falling: \n1V*(1+(R15/(R16+R17))) = 2.102V\nVsetpg_rising:\n1V*(1+((R15+R16)/R17)) = 2.311V"
Changed lines of the file:
@@
 P 12800 3300
 F 0 "R16" H 12650 3359 59  0000 L BNN
-F 1 "450K" H 12650 3170 59  0000 L BNN
+F 1 "453K" H 12650 3170 59  0000 L BNN
 F 2 "sprite:R0402" H 12800 3300 50  0001 C CNN
 F 3 "" H 12800 3300 50  0001 C CNN
@@
 1% REQ
 Text Notes 12550 9300 0    127  ~ 0
-All Caps 3.3V\nExcept C21 (16V)\nAll Passives 0402 \nAll Passives (5%)\nExcept R4, R15 - R21 (1%) \nSubject to Change\nR2, R11, R12, R22\nR7, R8\nC3\nMPPT Max efficiency:\nR7/(R7 + R8) = 87%\nVsetsd: \n1V*(1+R18/R19) = 2V\nVbat_term:\n(3/2)V*(1+R20/R21) = 2.7V\nVsetpg_falling: \n1V*(1+(R15/(R16+R17))) = 2.102V\nVsetpg_rising:\n1V*(1+((R15+R16)/R17)) = 2.311V
+All Caps 3.3V\nExcept C21 (16V)\nAll Passives 0402 \nAll Passives (5%)\nExcept R4, R15 - R21 (1%) \nSubject to Change\nR2, R11, R12, R22\nR7, R8\nC3\nMPPT Max efficiency:\nR7/(R7 + R8) = 87%\nVsetsd: \n1V*(1+R18/R19) = 2V\nVbat_term:\n(3/2)V*(1+R20/R21) = 2.7V\nVsetpg_falling: \n1V*(1+(R15/(R16+R17))) = 2.102V\nVsetpg_rising:\n1V*(1+((R15+R16)/R17)) = 2.312V
 Wire Notes Line
 	12200 9900 12200 4800

Commit message: Update schematic title block matter
Other:
- note removed: "Design By:"
- note removed: "Space Technologies at California\nstac.berkeley.edu"
Changed lines of the file:
@@
 EELAYER 26 0
 EELAYER END
-$Descr User 16797 11668
+$Descr B 17000 11000
 encoding utf-8
 Sheet 1 1
-Title ""
-Date ""
-Rev ""
-Comp ""
-Comment1 ""
+Title "PCBSat"
+Date "2018-06-17"
+Rev "v1.0"
+Comp "Space Technologies at California"
+Comment1 "stac.berkeley.edu"
 Comment2 ""
 Comment3 ""
@@
 $EndComp
 $Comp
-L sprite-eagle-import:A3L-LOC #FRAME1
-U 1 0 95E36ED37D0788B5
-P 900 10900
-F 0 "#FRAME1" H 900 10900 50  0001 C CNN
-F 1 "A3L-LOC" H 900 10900 50  0001 C CNN
-F 2 "" H 900 10900 50  0001 C CNN
-F 3 "" H 900 10900 50  0001 C CNN
-	1    900  10900
-	1    0    0    -1
-$EndComp
-$Comp
 L sprite-eagle-import:VCCINT #VCC05
 U 1 0 5B36E11081833CC9
@@
 Text Notes 8200 5200 0    170  ~ 0
 Torque Coils
-Text Notes 12300 10600 0    85   ~ 0
-Space Technologies at California\nstac.berkeley.edu
-Text Notes 12300 10200 0    102  ~ 0
-Design By:
 Text Notes 7500 1100 0    170  ~ 0
 Power
