File: kicad/final-sprite/sprite.sch (KiCad schematic (older format))
At the start: 62 parts, among them J1 M20-7910442R, U1 CC430F513X, U2 LSM9DS1, U3 SPRITETCXO_TCXO_7Z, U4 DRV8837, U5 ADP5092, U6 DRV8837, U7 DRV8837, X1 SPRITEPIN_SPRITE_PIN, X2 SPRITEPIN_SPRITE_PIN

Commit message: Fix inductor test points
Parts:
- added TP1: Test_Point, TestPoint:TestPoint_Pad_D1.0mm, symbol Connector:Test_Point
Connections:
- wire segments 267 -> 266
Changed lines of the file:
@@
 Text Notes 12200 4950 0    170  ~ 0
 Design Notes
-Text Notes 7900 9150 0    42   ~ 0
+Text Notes 8350 8750 0    42   ~ 0
 PCB Spiral Inductor\nLayers 2 and 3
 Wire Notes Line
@@
 $EndComp
 Wire Wire Line
-	8550 8850 8550 8800
-Wire Wire Line
 	8850 9750 8250 9750
 Wire Wire Line
@@
 NoConn ~ 2900 7550
 NoConn ~ 4700 2850
+$Comp
+L Connector:Test_Point TP1
+U 1 1 5B3A87A5
+P 8850 8950
+F 0 "TP1" H 8792 8977 50  0000 R CNN
+F 1 "Test_Point" H 8792 9068 50  0000 R CNN
+F 2 "TestPoint:TestPoint_Pad_D1.0mm" H 9050 8950 50  0001 C CNN
+F 3 "~" H 9050 8950 50  0001 C CNN
+	1    8850 8950
+	-1   0    0    -1
+$EndComp
+Connection ~ 8850 8950
 $EndSCHEMATC

Commit message: Fix size of R10
Parts:
- R10: value 750K -> 200k
Changed lines of the file:
@@
 P 8200 3750
 F 0 "R10" H 8050 3809 59  0000 L BNN
-F 1 "750K" H 8050 3620 59  0000 L BNN
+F 1 "200k" H 8050 3620 59  0000 L BNN
 F 2 "sprite:R0402" H 8200 3750 50  0001 C CNN
 F 3 "" H 8200 3750 50  0001 C CNN
