File: kicad/final-sprite-slot/sprite.sch (KiCad schematic (older format))
At the start: 64 parts, among them J1 M20-7910442R, U1 CC430F513X, U2 LSM9DS1, U3 SPRITETCXO_TCXO_7Z, U4 DRV8837, U5 ADP5092, U6 DRV8837, U7 DRV8837, X1 SPRITEPIN_SPRITE_PIN, X2 SPRITEPIN_SPRITE_PIN

Commit message: added in new super cap
Parts:
- removed C10: CPH3225A, CAPCP3225X100N, symbol CPH3225A:CPH3225A
- added B1: UMAC_UMAC, sprite:UMAC_UMAC, symbol sprite-eagle-import:UMAC_UMAC
- MK1: symbol sprite-rescue:Mounting_Hole-Mechanical -> Mechanical:Mounting_Hole
- TP1, TP2: symbol sprite-rescue:Test_Point-Connector -> Connector:Test_Point
Other:
- moved on the sheet: C17, D1, D2, D3, D4, R15, R16, R17, R18, R19, R20, R21

Commit message: moving some passives
Parts:
- MK1: symbol Mechanical:Mounting_Hole -> sprite-rescue:Mounting_Hole-Mechanical
- TP1, TP2: symbol Connector:Test_Point -> sprite-rescue:Test_Point-Connector
Changed lines of the file:
@@
 	800  4550 15700 4550
 $Comp
-L Mechanical:Mounting_Hole MK1
+L sprite-rescue:Mounting_Hole-Mechanical MK1
 U 1 1 5B277BCA
 P 13650 850
@@
 	9750 8700 10000 8700
 $Comp
-L Connector:Test_Point TP2
+L sprite-rescue:Test_Point-Connector TP2
 U 1 1 5B335398
 P 8250 8950
@@
 NoConn ~ 4700 2850
 $Comp
-L Connector:Test_Point TP1
+L sprite-rescue:Test_Point-Connector TP1
 U 1 1 5B3A87A5
 P 8850 8950
