File: kicad/final-sprite-respin/sprite.kicad_pcb (KiCad board)
At the start: 4 copper layers, 35 x 35 mm, 75 parts, among them J1 M20-7910442R, U1 CC430F513X, U2 LSM9DS1, U3 SPRITETCXO_TCXO_7Z, U4 DRV8837, U5 ADP5092, U6 DRV8837, U7 DRV8837, U8 TASC, U9 TASC, X1 SPRITEPIN_SPRITE_PIN, X2 SPRITEPIN_SPRITE_PIN

Commit message: final version
Other:
- outline, holes or cut-outs redrawn
- board text added: "NOTES: 1. MATERIAL: STANDARD 4-LAYER FR4 STACKUP, 0.031" OVERALL THICKNESS. 1 OZ COPPER ON ALL LAYERS. 2. FINISH: ELECTROLESS NICKEL IMMERSION GOLD (ENIG) 3. SOLDERMASK COLOR: LEAST EXPENSIVE OR BLACK. 4. TRIM COPPER AROUND BOARD EDGE AS NEEDED TO FABRICATE WITH STANDARD CAPABILITY. 5. MANUFACTURE WITH STANDARD CAPABILITIES. EXCEPT DESIGN RULES AS INDICATED."
- board text removed: "MECHANICAL EXCEPTION: ROUND EDGE HERE TO FABRICATE WITH STANDARD CAPABILITY."
- board text removed: "NOTES: 1. MATERIAL: STANDARD 4-LAYER FR4 STACKUP, 0.031" OVERALL THICKNESS. 1 OZ COPPER ON ALL LAYERS. 2. FINISH: ELECTROLESS NICKEL IMMERSION GOLD (ENIG) 3. VIAS: PLUG AND TENT ALL VIAS WITH SOLDERMASK. COLOR: LEAST EXPENSIVE OR BLACK. 4. TRIM COPPER AROUND BOARD EDGE AS NEEDED TO FABRICATE WITH STANDARD CAPABILITY. 5. MANUFACTURE WITH STANDARD CAPABILITIES. EXCEPT DESIGN RULES AS INDICATED."
- board text removed: "TRACE TO NPTH EXCEPTION: SHRINK PAD AS NEEDED TO FABRICATE WITH STANDARD CAPABILITY."
